Commit message: expand <gazebo> tag

File: urdf/macros_wheels.xacro (robot description, xacro)
@@ -6,8 +6,10 @@
     <xacro:macro name="populate_links" params="name_prefix x y z roll pitch yaw dx dy dz i:=1 count **template">
         <xacro:if value="${i &lt;= count}">
-            <link name="${name_prefix}${i}">
-                <pose>${x} ${y} ${z} ${roll} ${pitch} ${yaw}</pose>
-                <xacro:insert_block name="template" />
-            </link>
+            <gazebo>
+                <link name="${name_prefix}${i}">
+                    <pose>${x} ${y} ${z} ${roll} ${pitch} ${yaw}</pose>
+                    <xacro:insert_block name="template" />
+                </link>
+            </gazebo>
             <xacro:populate_links name_prefix="${name_prefix}" x="${x+dx}" y="${y+dy}" z="${z+dz}" roll="${roll}" pitch="${pitch}" yaw="${yaw}" dx="${dx}" dy="${dy}" dz="${dz}" i="${i+1}" count="${count}">
                 <template>
@@ -19,8 +21,10 @@
     <xacro:macro name="populate_joints" params="name_prefix type child_prefix i:=1 count **template">
         <xacro:if value="${i &lt;= count}">
-            <joint name="${name_prefix}${i}" type="${type}">
-                <child>${child_prefix}${i}</child>
-                <xacro:insert_block name="template" />
-            </joint>
+            <gazebo>
+                <joint name="${name_prefix}${i}" type="${type}">
+                    <child>${child_prefix}${i}</child>
+                    <xacro:insert_block name="template" />
+                </joint>
+            </gazebo>
             <xacro:populate_joints name_prefix="${name_prefix}" type="${type}" child_prefix="${child_prefix}" i="${i+1}" count="${count}">
                 <template>

Commit message: add friction coeff param

File: urdf/macros_wheels.xacro (robot description, xacro)
@@ -35,5 +35,5 @@
     </xacro:macro>
     <!-- wheel/axle/belt templates which can be used with above macros -->
-    <xacro:macro name="make_wheel_template" params="mass length radius">
+    <xacro:macro name="make_wheel_template" params="mass length radius mu">
         <inertial>
             <mass>${mass}</mass>
@@ -52,4 +52,12 @@
                 </cylinder>
             </geometry>
+            <surface>
+                <friction>
+                    <ode>
+                        <mu>${mu}</mu>
+                        <mu2>${mu}</mu2>
+                    </ode>
+                </friction>
+            </surface>
         </collision>
     </xacro:macro>
@@ -82,8 +90,8 @@
     </xacro:macro>
     <!-- macros for populating wheels/axles/belts with above macros and templates -->
-    <xacro:macro name="populate_wheels" params="name_prefix x:=0 y:=0 z:=0 roll:=0 pitch:=0 yaw:=0 dx:=0 dy:=0 dz:=0 mass length radius count">
+    <xacro:macro name="populate_wheels" params="name_prefix x:=0 y:=0 z:=0 roll:=0 pitch:=0 yaw:=0 dx:=0 dy:=0 dz:=0 mass length radius mu:=0.5 count">
         <xacro:populate_links name_prefix="${name_prefix}" x="${x}" y="${y}" z="${z}" roll="${roll}" pitch="${pitch}" yaw="${yaw}" dx="${dx}" dy="${dy}" dz="${dz}" count="${count}">
             <template>
-                <xacro:make_wheel_template mass="${mass}" length="${length}" radius="${radius}" />
+                <xacro:make_wheel_template mass="${mass}" length="${length}" radius="${radius}" mu="${mu}" />
             </template>
         </xacro:populate_links>

Commit message: add min_depth param to make contact more stable

File: urdf/macros_wheels.xacro (robot description, xacro)
@@ -35,5 +35,5 @@
     </xacro:macro>
     <!-- wheel/axle/belt templates which can be used with above macros -->
-    <xacro:macro name="make_wheel_template" params="mass length radius mu">
+    <xacro:macro name="make_wheel_template" params="mass length radius mu min_depth">
         <inertial>
             <mass>${mass}</mass>
@@ -59,4 +59,9 @@
                     </ode>
                 </friction>
+                <contact>
+                    <ode>
+                        <min_depth>${min_depth}</min_depth>
+                    </ode>
+                </contact>
             </surface>
         </collision>
@@ -90,8 +95,8 @@
     </xacro:macro>
     <!-- macros for populating wheels/axles/belts with above macros and templates -->
-    <xacro:macro name="populate_wheels" params="name_prefix x:=0 y:=0 z:=0 roll:=0 pitch:=0 yaw:=0 dx:=0 dy:=0 dz:=0 mass length radius mu:=0.5 count">
+    <xacro:macro name="populate_wheels" params="name_prefix x:=0 y:=0 z:=0 roll:=0 pitch:=0 yaw:=0 dx:=0 dy:=0 dz:=0 mass length radius mu:=0.5 min_depth:=0.01 count">
         <xacro:populate_links name_prefix="${name_prefix}" x="${x}" y="${y}" z="${z}" roll="${roll}" pitch="${pitch}" yaw="${yaw}" dx="${dx}" dy="${dy}" dz="${dz}" count="${count}">
             <template>
-                <xacro:make_wheel_template mass="${mass}" length="${length}" radius="${radius}" mu="${mu}" />
+                <xacro:make_wheel_template mass="${mass}" length="${length}" radius="${radius}" mu="${mu}" min_depth="${min_depth}" />
             </template>
         </xacro:populate_links>
