Commit message: change param names (sprocket -> sprocket_joint)

File: urdf/macros_track_gazebo.urdf.xacro (robot description, xacro)
@@ -64,9 +64,9 @@
     </xacro:macro>
     <!-- macro which expands to plugin definition -->
-    <xacro:macro name="make_track_plugin" params="name sprocket pitch_diameter length *pattern">
+    <xacro:macro name="make_track_plugin" params="name sprocket_joint pitch_diameter length *pattern">
         <gazebo>
             <plugin name="${name}" filename="libContinuousTrack.so">
                 <sprocket>
-                    <joint>${sprocket}</joint>
+                    <joint>${sprocket_joint}</joint>
                     <pitch_diameter>${pitch_diameter}</pitch_diameter>
                 </sprocket>
@@ -94,8 +94,8 @@
     </xacro:macro>
     <!-- main entry point: macro for making oval track by ContinuousTrack plugin -->
-    <xacro:macro name="make_track" params="name x:=0 y:=0 z:=0 roll:=0 pitch:=0 yaw:=0 mass length radius width parent sprocket pitch_diameter *pattern implicit_spring_damper:=1">
+    <xacro:macro name="make_track" params="name x:=0 y:=0 z:=0 roll:=0 pitch:=0 yaw:=0 mass length radius width parent sprocket_joint pitch_diameter *pattern implicit_spring_damper:=1">
         <xacro:populate_straight_segments name_prefix="${name}_straight_segment" x="${x - length / 2}" y="${y}" z="${z + radius}" roll="${roll}" pitch="${pitch}" yaw="${yaw}" dx="${length}" dz="${-2 * radius}" dpitch="${pi}" mass="${mass / 4}" size_x="${length}" size_y="${width}" size_z="${radius}" parent="${parent}" implicit_spring_damper="${implicit_spring_damper}" count="2" />
         <xacro:populate_arc_segments name_prefix="${name}_arc_segment" x="${x + length / 2}" y="${y}" z="${z + radius}" roll="${roll}" pitch="${pitch}" yaw="${yaw}" dx="${-length}" dz="${-2 * radius}" dpitch="${pi}" mass="${mass / 4}" length="${width}" radius="${radius}" parent="${parent}" implicit_spring_damper="${implicit_spring_damper}" count="2" />
-        <xacro:make_track_plugin name="${name}" sprocket="${sprocket}" pitch_diameter="${pitch_diameter}" length="${length}">
+        <xacro:make_track_plugin name="${name}" sprocket_joint="${sprocket_joint}" pitch_diameter="${pitch_diameter}" length="${length}">
             <xacro:insert_block name="pattern" />
         </xacro:make_track_plugin>

File: urdf/macros_track_simple_gazebo.urdf.xacro (robot description, xacro)
@@ -65,9 +65,9 @@
     </xacro:macro>
     <!-- macro which expands to simple plugin definition -->
-    <xacro:macro name="make_track_simple_plugin" params="name sprocket pitch_diameter">
+    <xacro:macro name="make_track_simple_plugin" params="name sprocket_joint pitch_diameter">
         <gazebo>
             <plugin name="${name}" filename="libContinuousTrackSimple.so">
                 <sprocket>
-                    <joint>${sprocket}</joint>
+                    <joint>${sprocket_joint}</joint>
                     <pitch_diameter>${pitch_diameter}</pitch_diameter>
                 </sprocket>
@@ -92,8 +92,8 @@
     </xacro:macro>
     <!-- main entry point: macro for making oval track by ContinuousTrackSimple plugin -->
-    <xacro:macro name="make_track_simple" params="name x:=0 y:=0 z:=0 roll:=0 pitch:=0 yaw:=0 mass length radius width parent sprocket pitch_diameter mu:=0.5 min_depth:=0.01 implicit_spring_damper:=1">
+    <xacro:macro name="make_track_simple" params="name x:=0 y:=0 z:=0 roll:=0 pitch:=0 yaw:=0 mass length radius width parent sprocket_joint pitch_diameter mu:=0.5 min_depth:=0.01 implicit_spring_damper:=1">
         <xacro:populate_straight_segments_simple name_prefix="${name}_straight_segment" x="${x}" y="${y}" z="${z + radius / 2}" roll="${roll}" pitch="${pitch}" yaw="${yaw}" dz="${-radius}" dpitch="${pi}" mass="${mass / 4}" size_x="${length}" size_y="${width}" size_z="${radius}" parent="${parent}" mu="${mu}" min_depth="${min_depth}" implicit_spring_damper="${implicit_spring_damper}" count="2" />
         <xacro:populate_arc_segments_simple name_prefix="${name}_arc_segment" x="${x + length / 2}" y="${y}" z="${z}" roll="${roll}" pitch="${pitch}" yaw="${yaw}" dx="${-length}" dpitch="${pi}" mass="${mass / 4}" length="${width}" radius="${radius}" parent="${parent}" mu="${mu}" min_depth="${min_depth}" implicit_spring_damper="${implicit_spring_damper}" count="2" />
-        <xacro:make_track_simple_plugin name="${name}" sprocket="${sprocket}" pitch_diameter="${pitch_diameter}" />
+        <xacro:make_track_simple_plugin name="${name}" sprocket_joint="${sprocket_joint}" pitch_diameter="${pitch_diameter}" />
     </xacro:macro>
 </robot>

Commit message: add make_box_element macro

File: urdf/macros_track_gazebo.urdf.xacro (robot description, xacro)
@@ -101,3 +101,10 @@
         </xacro:make_track_plugin>
     </xacro:macro>
+    <!-- macro which expands to box collision and visual. convenient when defining <pattern> in above macro -->
+    <xacro:macro name="make_box_element" params="pose:='0 0 0 0 0 0' size mu:=0.5 min_depth:=0.01 *material">
+        <xacro:make_box_collision pose="${pose}" size="${size}" mu="${mu}" min_depth="${min_depth}" />
+        <xacro:make_box_visual pose="${pose}" size="${size}">
+            <xacro:insert_block name="material" />
+        </xacro:make_box_visual>
+    </xacro:macro>
 </robot>
