Commit message: add make_track* macros & refactor

File: urdf/macros_common_gazebo.urdf.xacro (robot description, xacro)
@@ -99,3 +99,34 @@
         </visual>
     </xacro:macro>
+    <!-- macros for populating general links/joints -->
+    <xacro:macro name="populate_links" params="name_prefix x y z roll pitch yaw dx dy dz droll dpitch dyaw i:=1 count **template">
+        <xacro:if value="${i &lt;= count}">
+            <gazebo>
+                <link name="${name_prefix}${i}">
+                    <pose>${x} ${y} ${z} ${roll} ${pitch} ${yaw}</pose>
+                    <xacro:insert_block name="template" />
+                </link>
+            </gazebo>
+            <xacro:populate_links name_prefix="${name_prefix}" x="${x+dx}" y="${y+dy}" z="${z+dz}" roll="${roll+droll}" pitch="${pitch+dpitch}" yaw="${yaw+dyaw}" dx="${dx}" dy="${dy}" dz="${dz}" droll="${droll}" dpitch="${dpitch}" dyaw="${dyaw}" i="${i+1}" count="${count}">
+                <template>
+                    <xacro:insert_block name="template" />
+                </template>
+            </xacro:populate_links>
+        </xacro:if>
+    </xacro:macro>
+    <xacro:macro name="populate_joints" params="name_prefix type child_prefix i:=1 count **template">
+        <xacro:if value="${i &lt;= count}">
+            <gazebo>
+                <joint name="${name_prefix}${i}" type="${type}">
+                    <child>${child_prefix}${i}</child>
+                    <xacro:insert_block name="template" />
+                </joint>
+            </gazebo>
+            <xacro:populate_joints name_prefix="${name_prefix}" type="${type}" child_prefix="${child_prefix}" i="${i+1}" count="${count}">
+                <template>
+                    <xacro:insert_block name="template" />
+                </template>
+            </xacro:populate_joints>
+        </xacro:if>
+    </xacro:macro>
 </robot>

Commit message: use outer-scope properties

File: urdf/macros_common_gazebo.urdf.xacro (robot description, xacro)
@@ -1,5 +1,5 @@
 <robot xmlns:xacro="http://www.ros.org/wiki/xacro">
     <!-- macros which expand to inertial/collision/visual -->
-    <xacro:macro name="make_cylinder_inertial" params="pose:='0 0 0 0 0 0' mass length radius">
+    <xacro:macro name="make_cylinder_inertial" params="pose:=^|'0 0 0 0 0 0' mass:=^ length:=^ radius:=^">
         <inertial>
             <pose>${pose}</pose>
@@ -15,5 +15,5 @@
         </inertial>
     </xacro:macro>
-    <xacro:macro name="make_cylinder_collision" params="name:='collision' pose:='0 0 0 0 0 0' length radius mu:=0.5 min_depth:=0.01">
+    <xacro:macro name="make_cylinder_collision" params="name:='collision' pose:=^|'0 0 0 0 0 0' length:=^ radius:=^ mu:=^|0.5 min_depth:=^|0.01">
         <collision name="${name}">
             <pose>${pose}</pose>
@@ -39,5 +39,5 @@
         </collision>
     </xacro:macro>
-    <xacro:macro name="make_cylinder_visual" params="name:='visual' pose:='0 0 0 0 0 0' length radius *material">
+    <xacro:macro name="make_cylinder_visual" params="name:='visual' pose:=^|'0 0 0 0 0 0' length:=^ radius:=^ *material">
         <visual name="${name}">
             <pose>${pose}</pose>
@@ -51,5 +51,5 @@
         </visual>
     </xacro:macro>
-    <xacro:macro name="make_box_inertial" params="pose:='0 0 0 0 0 0' mass size_x size_y size_z">
+    <xacro:macro name="make_box_inertial" params="pose:=^|'0 0 0 0 0 0' mass:=^ size_x:=^ size_y:=^ size_z:=^">
         <inertial>
             <pose>${pose}</pose>
@@ -65,5 +65,5 @@
         </inertial>
     </xacro:macro>
-    <xacro:macro name="make_box_collision" params="name:='collision' pose:='0 0 0 0 0 0' size mu:=0.5 min_depth:=0.01">
+    <xacro:macro name="make_box_collision" params="name:='collision' pose:=^|'0 0 0 0 0 0' size:=^ mu:=^|0.5 min_depth:=^|0.01">
         <collision name="${name}">
             <pose>${pose}</pose>
@@ -88,5 +88,5 @@
         </collision>
     </xacro:macro>
-    <xacro:macro name="make_box_visual" params="name:='visual' pose:='0 0 0 0 0 0' size *material">
+    <xacro:macro name="make_box_visual" params="name:='visual' pose:=^|'0 0 0 0 0 0' size:=^ *material">
         <visual name="${name}">
             <pose>${pose}</pose>
@@ -100,5 +100,5 @@
     </xacro:macro>
     <!-- macros for populating general links/joints -->
-    <xacro:macro name="populate_links" params="name_prefix x y z roll pitch yaw dx dy dz droll dpitch dyaw i:=1 count **template">
+    <xacro:macro name="populate_links" params="name_prefix:=^ x:=^|0 y:=^|0 z:=^|0 roll:=^|0 pitch:=^|0 yaw:=^|0 dx:=^|0 dy:=^|0 dz:=^|0 droll:=^|0 dpitch:=^|0 dyaw:=^|0 i:=1 count:=^ **template">
         <xacro:if value="${i &lt;= count}">
             <gazebo>
@@ -108,5 +108,5 @@
                 </link>
             </gazebo>
-            <xacro:populate_links name_prefix="${name_prefix}" x="${x+dx}" y="${y+dy}" z="${z+dz}" roll="${roll+droll}" pitch="${pitch+dpitch}" yaw="${yaw+dyaw}" dx="${dx}" dy="${dy}" dz="${dz}" droll="${droll}" dpitch="${dpitch}" dyaw="${dyaw}" i="${i+1}" count="${count}">
+            <xacro:populate_links x="${x+dx}" y="${y+dy}" z="${z+dz}" roll="${roll+droll}" pitch="${pitch+dpitch}" yaw="${yaw+dyaw}" i="${i+1}">
                 <template>
                     <xacro:insert_block name="template" />
@@ -115,5 +115,5 @@
         </xacro:if>
     </xacro:macro>
-    <xacro:macro name="populate_joints" params="name_prefix type child_prefix i:=1 count **template">
+    <xacro:macro name="populate_joints" params="name_prefix:=^ type:=^ child_prefix:=^ i:=1 count:=^ **template">
         <xacro:if value="${i &lt;= count}">
             <gazebo>
@@ -123,5 +123,5 @@
                 </joint>
             </gazebo>
-            <xacro:populate_joints name_prefix="${name_prefix}" type="${type}" child_prefix="${child_prefix}" i="${i+1}" count="${count}">
+            <xacro:populate_joints i="${i+1}">
                 <template>
                     <xacro:insert_block name="template" />

File: urdf/macros_track_gazebo.urdf.xacro (robot description, xacro)
@@ -7,8 +7,8 @@
     <xacro:include filename="macros_common_gazebo.urdf.xacro" />
     <!-- trajectory segment templates which can be used with common population macros -->
-    <xacro:macro name="make_straight_segment_link_template" params="mass size_x size_y size_z">
-        <xacro:make_box_inertial pose="${size_x / 2} 0 0 0 0 0" mass="${mass}" size_x="${size_x}" size_y="${size_y}" size_z="${size_z}" />
+    <xacro:macro name="make_straight_segment_link_template" params="mass:=^ size_x:=^ size_y:=^ size_z:=^">
+        <xacro:make_box_inertial pose="${size_x / 2} 0 0 0 0 0" />
     </xacro:macro>
-    <xacro:macro name="make_straight_segment_joint_template" params="parent implicit_spring_damper">
+    <xacro:macro name="make_straight_segment_joint_template" params="parent:=^ implicit_spring_damper:=^|1">
         <parent>${parent}</parent>
         <axis>
@@ -22,8 +22,8 @@
         </physics>
     </xacro:macro>
-    <xacro:macro name="make_arc_segment_link_template" params="mass length radius">
-        <xacro:make_cylinder_inertial pose="0 0 ${-radius} ${pi / 2} 0 0" mass="${mass}" length="${length}" radius="${radius}" />
+    <xacro:macro name="make_arc_segment_link_template" params="mass:=^ length:=^ radius:=^">
+        <xacro:make_cylinder_inertial pose="0 0 ${-radius} ${pi / 2} 0 0" />
     </xacro:macro>
-    <xacro:macro name="make_arc_segment_joint_template" params="parent radius implicit_spring_damper">
+    <xacro:macro name="make_arc_segment_joint_template" params="parent:=^ radius:=^ implicit_spring_damper:=^|1">
         <parent>${parent}</parent>
         <pose>0 0 ${-radius} 0 0 0</pose>
@@ -39,30 +39,30 @@
     </xacro:macro>
     <!-- macros for populating trajectory segments with common population macros and above templates -->
-    <xacro:macro name="populate_straight_segments" params="name_prefix x:=0 y:=0 z:=0 roll:=0 pitch:=0 yaw:=0 dx:=0 dy:=0 dz:=0 droll:=0 dpitch:=0 dyaw:=0 mass size_x size_y size_z parent implicit_spring_damper:=1 count">
-        <xacro:populate_links name_prefix="${name_prefix}_link" x="${x}" y="${y}" z="${z}" roll="${roll}" pitch="${pitch}" yaw="${yaw}" dx="${dx}" dy="${dy}" dz="${dz}" droll="${droll}" dpitch="${dpitch}" dyaw="${dyaw}" count="${count}">
+    <xacro:macro name="populate_straight_segments" params="name_prefix:=^ x:=^|0 y:=^|0 z:=^|0 roll:=^|0 pitch:=^|0 yaw:=^|0 dx:=^|0 dy:=^|0 dz:=^|0 droll:=^|0 dpitch:=^|0 dyaw:=^|0 mass:=^ size_x:=^ size_y:=^ size_z:=^ parent:=^ implicit_spring_damper:=^|1 count:=^">
+        <xacro:populate_links name_prefix="${name_prefix}_link">
             <template>
-                <xacro:make_straight_segment_link_template mass="${mass}" size_x="${size_x}" size_y="${size_y}" size_z="${size_z}" />
+                <xacro:make_straight_segment_link_template />
             </template>
         </xacro:populate_links>
-        <xacro:populate_joints name_prefix="${name_prefix}_joint" type="prismatic" child_prefix="${name_prefix}_link" count="${count}">
+        <xacro:populate_joints name_prefix="${name_prefix}_joint" type="prismatic" child_prefix="${name_prefix}_link">
             <template>
-                <xacro:make_straight_segment_joint_template parent="${parent}" implicit_spring_damper="${implicit_spring_damper}" />
+                <xacro:make_straight_segment_joint_template />
             </template>
         </xacro:populate_joints>
     </xacro:macro>
-    <xacro:macro name="populate_arc_segments" params="name_prefix x:=0 y:=0 z:=0 roll:=0 pitch:=0 yaw:=0 dx:=0 dy:=0 dz:=0 droll:=0 dpitch:=0 dyaw:=0 mass length radius parent implicit_spring_damper:=1 count">
-        <xacro:populate_links name_prefix="${name_prefix}_link" x="${x}" y="${y}" z="${z}" roll="${roll}" pitch="${pitch}" yaw="${yaw}" dx="${dx}" dy="${dy}" dz="${dz}" droll="${droll}" dpitch="${dpitch}" dyaw="${dyaw}" count="${count}">
+    <xacro:macro name="populate_arc_segments" params="name_prefix:=^ x:=^|0 y:=^|0 z:=^|0 roll:=^|0 pitch:=^|0 yaw:=^|0 dx:=^|0 dy:=^|0 dz:=^|0 droll:=^|0 dpitch:=^|0 dyaw:=^|0 mass:=^ length:=^ radius:=^ parent:=^ implicit_spring_damper:=^|1 count:=^">
+        <xacro:populate_links name_prefix="${name_prefix}_link">
             <template>
-                <xacro:make_arc_segment_link_template mass="${mass}" length="${length}" radius="${radius}" />
+                <xacro:make_arc_segment_link_template />
             </template>
         </xacro:populate_links>
-        <xacro:populate_joints name_prefix="${name_prefix}_joint" type="revolute" child_prefix="${name_prefix}_link" count="${count}">
+        <xacro:populate_joints name_prefix="${name_prefix}_joint" type="revolute" child_prefix="${name_prefix}_link">
             <template>
-                <xacro:make_arc_segment_joint_template parent="${parent}" radius="${radius}" implicit_spring_damper="${implicit_spring_damper}" />
+                <xacro:make_arc_segment_joint_template />
             </template>
         </xacro:populate_joints>
     </xacro:macro>
     <!-- macro which expands to plugin definition -->
-    <xacro:macro name="make_track_plugin" params="name sprocket_joint pitch_diameter length *pattern">
+    <xacro:macro name="make_track_plugin" params="name sprocket_joint:=^ pitch_diameter:=^ length:=^ *pattern">
         <gazebo>
             <plugin name="${name}" filename="libContinuousTrack.so">
@@ -94,15 +94,15 @@
     </xacro:macro>
     <!-- main entry point: macro for making oval track by ContinuousTrack plugin -->
-    <xacro:macro name="make_track" params="name x:=0 y:=0 z:=0 roll:=0 pitch:=0 yaw:=0 mass length radius width parent sprocket_joint pitch_diameter *pattern implicit_spring_damper:=1">
-        <xacro:populate_straight_segments name_prefix="${name}_straight_segment" x="${x - length / 2}" y="${y}" z="${z + radius}" roll="${roll}" pitch="${pitch}" yaw="${yaw}" dx="${length}" dz="${-2 * radius}" dpitch="${pi}" mass="${mass / 4}" size_x="${length}" size_y="${width}" size_z="${radius}" parent="${parent}" implicit_spring_damper="${implicit_spring_damper}" count="2" />
-        <xacro:populate_arc_segments name_prefix="${name}_arc_segment" x="${x + length / 2}" y="${y}" z="${z + radius}" roll="${roll}" pitch="${pitch}" yaw="${yaw}" dx="${-length}" dz="${-2 * radius}" dpitch="${pi}" mass="${mass / 4}" length="${width}" radius="${radius}" parent="${parent}" implicit_spring_damper="${implicit_spring_damper}" count="2" />
-        <xacro:make_track_plugin name="${name}" sprocket_joint="${sprocket_joint}" pitch_diameter="${pitch_diameter}" length="${length}">
+    <xacro:macro name="make_track" params="name x:=^|0 y:=^|0 z:=^|0 roll:=^|0 pitch:=^|0 yaw:=^|0 mass:=^ length:=^ radius:=^ width:=^ parent:=^ sprocket_joint:=^ pitch_diameter:=^ *pattern implicit_spring_damper:=^|1">
+        <xacro:populate_straight_segments name_prefix="${name}_straight_segment" x="${x - length / 2}" z="${z + radius}" dx="${length}" dz="${-2 * radius}" dpitch="${pi}" mass="${mass / 4}" size_x="${length}" size_y="${width}" size_z="${radius}" count="2" />
+        <xacro:populate_arc_segments name_prefix="${name}_arc_segment" x="${x + length / 2}" z="${z + radius}" dx="${-length}" dz="${-2 * radius}" dpitch="${pi}" mass="${mass / 4}" length="${width}" count="2" />
+        <xacro:make_track_plugin name="${name}">
             <xacro:insert_block name="pattern" />
         </xacro:make_track_plugin>
     </xacro:macro>
     <!-- macro which expands to box collision and visual. convenient when defining <pattern> in above macro -->
-    <xacro:macro name="make_box_element" params="pose:='0 0 0 0 0 0' size mu:=0.5 min_depth:=0.01 *material">
-        <xacro:make_box_collision pose="${pose}" size="${size}" mu="${mu}" min_depth="${min_depth}" />
-        <xacro:make_box_visual pose="${pose}" size="${size}">
+    <xacro:macro name="make_box_element" params="pose:=^|'0 0 0 0 0 0' size:=^ mu:=^|0.5 min_depth:=^|0.01 *material">
+        <xacro:make_box_collision />
+        <xacro:make_box_visual>
             <xacro:insert_block name="material" />
         </xacro:make_box_visual>
