Commit message: use outer-scope properties

File: urdf/macros_track_simple_gazebo.urdf.xacro (robot description, xacro)
@@ -7,14 +7,12 @@
     <xacro:include filename="macros_common_gazebo.urdf.xacro" />
     <!-- track segment templates which can be used with common population macros -->
-    <xacro:macro name="make_straight_segment_simple_link_template" params="mass size_x size_y size_z mu min_depth enable_visual *material">
-        <xacro:make_box_inertial mass="${mass}" size_x="${size_x}" size_y="${size_y}" size_z="${size_z}" />
-        <xacro:make_box_collision size="${size_x} ${size_y} ${size_z}" mu="${mu}" min_depth="${min_depth}" />
-        <xacro:if value="${enable_visual}">
-            <xacro:make_box_visual size="${size_x} ${size_y} ${size_z}">
-                <xacro:insert_block name="material" />
-            </xacro:make_box_visual>
-        </xacro:if>
+    <xacro:macro name="make_straight_segment_simple_link_template" params="mass:=^ size_x:=^ size_y:=^ size_z:=^ mu:=^|0.5 min_depth:=^|0.01 *material">
+        <xacro:make_box_inertial  />
+        <xacro:make_box_collision size="${size_x} ${size_y} ${size_z}" />
+        <xacro:make_box_visual size="${size_x} ${size_y} ${size_z}">
+            <xacro:insert_block name="material" />
+        </xacro:make_box_visual>
     </xacro:macro>
-    <xacro:macro name="make_straight_segment_simple_joint_template" params="parent implicit_spring_damper">
+    <xacro:macro name="make_straight_segment_simple_joint_template" params="parent:=^ implicit_spring_damper:=^|1">
         <parent>${parent}</parent>
         <axis>
@@ -28,14 +26,12 @@
         </physics>
     </xacro:macro>
-    <xacro:macro name="make_arc_segment_simple_link_template" params="mass length radius mu min_depth enable_visual *material">
-        <xacro:make_cylinder_inertial pose="0 0 0 ${pi / 2} 0 0" mass="${mass}" length="${length}" radius="${radius}" />
-        <xacro:make_cylinder_collision pose="0 0 0 ${pi / 2} 0 0" length="${length}" radius="${radius}" mu="${mu}" min_depth="${min_depth}" />
-        <xacro:if value="${enable_visual}">
-            <xacro:make_cylinder_visual pose="0 0 0 ${pi / 2} 0 0" length="${length}" radius="${radius}">
-                <xacro:insert_block name="material" />
-            </xacro:make_cylinder_visual>
-        </xacro:if>
+    <xacro:macro name="make_arc_segment_simple_link_template" params="mass:=^ length:=^ radius:=^ mu:=^|0.5 min_depth:=^|0.5 *material">
+        <xacro:make_cylinder_inertial pose="0 0 0 ${pi / 2} 0 0" />
+        <xacro:make_cylinder_collision pose="0 0 0 ${pi / 2} 0 0" />
+        <xacro:make_cylinder_visual pose="0 0 0 ${pi / 2} 0 0">
+            <xacro:insert_block name="material" />
+        </xacro:make_cylinder_visual>
     </xacro:macro>
-    <xacro:macro name="make_arc_segment_simple_joint_template" params="parent implicit_spring_damper">
+    <xacro:macro name="make_arc_segment_simple_joint_template" params="parent:=^ implicit_spring_damper:=^|1">
         <parent>${parent}</parent>
         <axis>
@@ -50,64 +46,34 @@
     </xacro:macro>
     <!-- macros for populating segments with common population macros and templates -->
-    <xacro:macro name="populate_straight_segments_simple_no_visual" params="name_prefix x:=0 y:=0 z:=0 roll:=0 pitch:=0 yaw:=0 dx:=0 dy:=0 dz:=0 droll:=0 dpitch:=0 dyaw:=0 mass size_x size_y size_z parent mu:=0.5 min_depth:=0.01 implicit_spring_damper:=1 count">
-        <xacro:populate_links name_prefix="${name_prefix}_link" x="${x}" y="${y}" z="${z}" roll="${roll}" pitch="${pitch}" yaw="${yaw}" dx="${dx}" dy="${dy}" dz="${dz}" droll="${droll}" dpitch="${dpitch}" dyaw="${dyaw}" count="${count}">
+    <xacro:macro name="populate_straight_segments_simple" params="name_prefix:=^ x:=^|0 y:=^|0 z:=^|0 roll:=^|0 pitch:=^|0 yaw:=^|0 dx:=^|0 dy:=^|0 dz:=^|0 droll:=^|0 dpitch:=^|0 dyaw:=^|0 mass:=^ size_x:=^ size_y:=^ size_z:=^ parent:=^ mu:=^|0.5 min_depth:=^|0.01 implicit_spring_damper:=^|1 *material count:=^">
+        <xacro:populate_links name_prefix="${name_prefix}_link">
             <template>
-                <xacro:make_straight_segment_simple_link_template mass="${mass}" size_x="${size_x}" size_y="${size_y}" size_z="${size_z}" mu="${mu}" min_depth="${min_depth}" enable_visual="0">
-                    <dummy />
-                </xacro:make_straight_segment_simple_link_template>
-            </template>
-        </xacro:populate_links>
-        <xacro:populate_joints name_prefix="${name_prefix}_joint" type="prismatic" child_prefix="${name_prefix}_link" count="${count}">
-            <template>
-                <xacro:make_straight_segment_simple_joint_template parent="${parent}" implicit_spring_damper="${implicit_spring_damper}" />
-            </template>
-        </xacro:populate_joints>
-    </xacro:macro>
-    <!-- with visual -->
-    <xacro:macro name="populate_straight_segments_simple" params="name_prefix x:=0 y:=0 z:=0 roll:=0 pitch:=0 yaw:=0 dx:=0 dy:=0 dz:=0 droll:=0 dpitch:=0 dyaw:=0 mass size_x size_y size_z parent mu:=0.5 min_depth:=0.01 implicit_spring_damper:=1 *material count">
-        <xacro:populate_links name_prefix="${name_prefix}_link" x="${x}" y="${y}" z="${z}" roll="${roll}" pitch="${pitch}" yaw="${yaw}" dx="${dx}" dy="${dy}" dz="${dz}" droll="${droll}" dpitch="${dpitch}" dyaw="${dyaw}" count="${count}">
-            <template>
-                <xacro:make_straight_segment_simple_link_template mass="${mass}" size_x="${size_x}" size_y="${size_y}" size_z="${size_z}" mu="${mu}" min_depth="${min_depth}" enable_visual="1">
+                <xacro:make_straight_segment_simple_link_template>
                     <xacro:insert_block name="material" />
                 </xacro:make_straight_segment_simple_link_template>
             </template>
         </xacro:populate_links>
-        <xacro:populate_joints name_prefix="${name_prefix}_joint" type="prismatic" child_prefix="${name_prefix}_link" count="${count}">
+        <xacro:populate_joints name_prefix="${name_prefix}_joint" type="prismatic" child_prefix="${name_prefix}_link">
             <template>
-                <xacro:make_straight_segment_simple_joint_template parent="${parent}" implicit_spring_damper="${implicit_spring_damper}" />
+                <xacro:make_straight_segment_simple_joint_template />
             </template>
         </xacro:populate_joints>
     </xacro:macro>
-    <xacro:macro name="populate_arc_segments_simple_no_visual" params="name_prefix x:=0 y:=0 z:=0 roll:=0 pitch:=0 yaw:=0 dx:=0 dy:=0 dz:=0 droll:=0 dpitch:=0 dyaw:=0 mass length radius parent mu:=0.5 min_depth:=0.01 implicit_spring_damper:=1 count">
-        <xacro:populate_links name_prefix="${name_prefix}_link" x="${x}" y="${y}" z="${z}" roll="${roll}" pitch="${pitch}" yaw="${yaw}" dx="${dx}" dy="${dy}" dz="${dz}" droll="${droll}" dpitch="${dpitch}" dyaw="${dyaw}" count="${count}">
+    <xacro:macro name="populate_arc_segments_simple" params="name_prefix:=^ x:=^|0 y:=^|0 z:=^|0 roll:=^|0 pitch:=^|0 yaw:=^|0 dx:=^|0 dy:=^|0 dz:=^|0 droll:=^|0 dpitch:=^|0 dyaw:=^|0 mass:=^ length:=^ radius:=^ parent:=^ mu:=^|0.5 min_depth:=^|0.01 implicit_spring_damper:=^|1 *material count:=^">
+        <xacro:populate_links name_prefix="${name_prefix}_link">
             <template>
-                <xacro:make_arc_segment_simple_link_template mass="${mass}" length="${length}" radius="${radius}" mu="${mu}" min_depth="${min_depth}" enable_visual="0">
-                    <dummy />
-                </xacro:make_arc_segment_simple_link_template>
-            </template>
-        </xacro:populate_links>
-        <xacro:populate_joints name_prefix="${name_prefix}_joint" type="revolute" child_prefix="${name_prefix}_link" count="${count}">
-            <template>
-                <xacro:make_arc_segment_simple_joint_template parent="${parent}" implicit_spring_damper="${implicit_spring_damper}" />
-            </template>
-        </xacro:populate_joints>
-    </xacro:macro>
-    <!-- with visual -->
-    <xacro:macro name="populate_arc_segments_simple" params="name_prefix x:=0 y:=0 z:=0 roll:=0 pitch:=0 yaw:=0 dx:=0 dy:=0 dz:=0 droll:=0 dpitch:=0 dyaw:=0 mass length radius parent mu:=0.5 min_depth:=0.01 implicit_spring_damper:=1 *material count">
-        <xacro:populate_links name_prefix="${name_prefix}_link" x="${x}" y="${y}" z="${z}" roll="${roll}" pitch="${pitch}" yaw="${yaw}" dx="${dx}" dy="${dy}" dz="${dz}" droll="${droll}" dpitch="${dpitch}" dyaw="${dyaw}" count="${count}">
-            <template>
-                <xacro:make_arc_segment_simple_link_template mass="${mass}" length="${length}" radius="${radius}" mu="${mu}" min_depth="${min_depth}" enable_visual="1">
+                <xacro:make_arc_segment_simple_link_template >
                     <xacro:insert_block name="material" />
                 </xacro:make_arc_segment_simple_link_template>
             </template>
         </xacro:populate_links>
-        <xacro:populate_joints name_prefix="${name_prefix}_joint" type="revolute" child_prefix="${name_prefix}_link" count="${count}">
+        <xacro:populate_joints name_prefix="${name_prefix}_joint" type="revolute" child_prefix="${name_prefix}_link">
             <template>
-                <xacro:make_arc_segment_simple_joint_template parent="${parent}" implicit_spring_damper="${implicit_spring_damper}" />
+                <xacro:make_arc_segment_simple_joint_template />
             </template>
         </xacro:populate_joints>
     </xacro:macro>
     <!-- macro which expands to simple plugin definition -->
-    <xacro:macro name="make_track_simple_plugin" params="name sprocket_joint pitch_diameter">
+    <xacro:macro name="make_track_simple_plugin" params="name sprocket_joint:=^ pitch_diameter:=^">
         <gazebo>
             <plugin name="${name}" filename="libContinuousTrackSimple.so">
@@ -136,18 +102,12 @@
     </xacro:macro>
     <!-- main entry point: macro for making oval track by ContinuousTrackSimple plugin -->
-    <xacro:macro name="make_track_simple_no_visual" params="name x:=0 y:=0 z:=0 roll:=0 pitch:=0 yaw:=0 mass length radius width parent sprocket_joint pitch_diameter mu:=0.5 min_depth:=0.01 implicit_spring_damper:=1">
-        <xacro:populate_straight_segments_simple_no_visual name_prefix="${name}_straight_segment" x="${x}" y="${y}" z="${z + radius / 2}" roll="${roll}" pitch="${pitch}" yaw="${yaw}" dz="${-radius}" dpitch="${pi}" mass="${mass / 4}" size_x="${length}" size_y="${width}" size_z="${radius}" parent="${parent}" mu="${mu}" min_depth="${min_depth}" implicit_spring_damper="${implicit_spring_damper}" count="2" />
-        <xacro:populate_arc_segments_simple_no_visual name_prefix="${name}_arc_segment" x="${x + length / 2}" y="${y}" z="${z}" roll="${roll}" pitch="${pitch}" yaw="${yaw}" dx="${-length}" dpitch="${pi}" mass="${mass / 4}" length="${width}" radius="${radius}" parent="${parent}" mu="${mu}" min_depth="${min_depth}" implicit_spring_damper="${implicit_spring_damper}" count="2" />
-        <xacro:make_track_simple_plugin name="${name}" sprocket_joint="${sprocket_joint}" pitch_diameter="${pitch_diameter}" />
-    </xacro:macro>
-    <!-- with visual -->
-    <xacro:macro name="make_track_simple" params="name x:=0 y:=0 z:=0 roll:=0 pitch:=0 yaw:=0 mass length radius width parent sprocket_joint pitch_diameter mu:=0.5 min_depth:=0.01 implicit_spring_damper:=1 *material">
-        <xacro:populate_straight_segments_simple name_prefix="${name}_straight_segment" x="${x}" y="${y}" z="${z + radius / 2}" roll="${roll}" pitch="${pitch}" yaw="${yaw}" dz="${-radius}" dpitch="${pi}" mass="${mass / 4}" size_x="${length}" size_y="${width}" size_z="${radius}" parent="${parent}" mu="${mu}" min_depth="${min_depth}" implicit_spring_damper="${implicit_spring_damper}" count="2">
+    <xacro:macro name="make_track_simple" params="name x:=^|0 y:=^|0 z:=^|0 roll:=^|0 pitch:=^|0 yaw:=^|0 mass:=^ length:=^ radius:=^ width:=^ parent:=^ sprocket_joint:=^ pitch_diameter:=^ mu:=^|0.5 min_depth:=^|0.01 implicit_spring_damper:=^|1 *material">
+        <xacro:populate_straight_segments_simple name_prefix="${name}_straight_segment" z="${z + radius / 2}" dz="${-radius}" dpitch="${pi}" mass="${mass / 4}" size_x="${length}" size_y="${width}" size_z="${radius}" count="2">
             <xacro:insert_block name="material" />
         </xacro:populate_straight_segments_simple>
-        <xacro:populate_arc_segments_simple name_prefix="${name}_arc_segment" x="${x + length / 2}" y="${y}" z="${z}" roll="${roll}" pitch="${pitch}" yaw="${yaw}" dx="${-length}" dpitch="${pi}" mass="${mass / 4}" length="${width}" radius="${radius}" parent="${parent}" mu="${mu}" min_depth="${min_depth}" implicit_spring_damper="${implicit_spring_damper}" count="2">
+        <xacro:populate_arc_segments_simple name_prefix="${name}_arc_segment" x="${x + length / 2}" dx="${-length}" dpitch="${pi}" mass="${mass / 4}" length="${width}" count="2">
             <xacro:insert_block name="material" />
         </xacro:populate_arc_segments_simple>
-        <xacro:make_track_simple_plugin name="${name}" sprocket_joint="${sprocket_joint}" pitch_diameter="${pitch_diameter}" />
+        <xacro:make_track_simple_plugin name="${name}" />
     </xacro:macro>
 </robot>

Commit message: 0-based indexing

File: urdf/macros_common_gazebo.urdf.xacro (robot description, xacro)
@@ -100,6 +100,6 @@
     </xacro:macro>
     <!-- macros for populating general links/joints -->
-    <xacro:macro name="populate_links" params="name_prefix:=^ x:=^|0 y:=^|0 z:=^|0 roll:=^|0 pitch:=^|0 yaw:=^|0 dx:=^|0 dy:=^|0 dz:=^|0 droll:=^|0 dpitch:=^|0 dyaw:=^|0 i:=1 count:=^ **template">
-        <xacro:if value="${i &lt;= count}">
+    <xacro:macro name="populate_links" params="name_prefix:=^ x:=^|0 y:=^|0 z:=^|0 roll:=^|0 pitch:=^|0 yaw:=^|0 dx:=^|0 dy:=^|0 dz:=^|0 droll:=^|0 dpitch:=^|0 dyaw:=^|0 i:=0 count:=^ **template">
+        <xacro:if value="${i &lt; count}">
             <gazebo>
                 <link name="${name_prefix}${i}">
@@ -115,6 +115,6 @@
         </xacro:if>
     </xacro:macro>
-    <xacro:macro name="populate_joints" params="name_prefix:=^ type:=^ child_prefix:=^ i:=1 count:=^ **template">
-        <xacro:if value="${i &lt;= count}">
+    <xacro:macro name="populate_joints" params="name_prefix:=^ type:=^ child_prefix:=^ i:=0 count:=^ **template">
+        <xacro:if value="${i &lt; count}">
             <gazebo>
                 <joint name="${name_prefix}${i}" type="${type}">

File: urdf/macros_track_gazebo.urdf.xacro (robot description, xacro)
@@ -73,4 +73,12 @@
                 <trajectory>
                     <segment>
+                        <joint>${name}_straight_segment_joint0</joint>
+                        <end_position>${length}</end_position>
+                    </segment>
+                    <segment>
+                        <joint>${name}_arc_segment_joint0</joint>
+                        <end_position>${pi}</end_position>
+                    </segment>
+                    <segment>
                         <joint>${name}_straight_segment_joint1</joint>
                         <end_position>${length}</end_position>
@@ -78,12 +86,4 @@
                     <segment>
                         <joint>${name}_arc_segment_joint1</joint>
-                        <end_position>${pi}</end_position>
-                    </segment>
-                    <segment>
-                        <joint>${name}_straight_segment_joint2</joint>
-                        <end_position>${length}</end_position>
-                    </segment>
-                    <segment>
-                        <joint>${name}_arc_segment_joint2</joint>
                         <end_position>${pi}</end_position>
                     </segment>

File: urdf/macros_track_simple_gazebo.urdf.xacro (robot description, xacro)
@@ -74,6 +74,6 @@
         </xacro:populate_joints>
     </xacro:macro>
-    <xacro:macro name="populate_arc_segments_simple_for_plugin" params="name_prefix:=^ pitch_diameter:=^ i:=1 count=^">
-        <xacro:if value="${i &lt;= count}">
+    <xacro:macro name="populate_arc_segments_simple_for_plugin" params="name_prefix:=^ pitch_diameter:=^ i:=0 count=^">
+        <xacro:if value="${i &lt; count}">
             <segment>
                 <joint>${name_prefix}${i}</joint>
@@ -93,15 +93,15 @@
                 <track>
                     <segment>
+                        <joint>${name}_straight_segment_joint0</joint>
+                    </segment>
+                    <segment>
+                        <joint>${name}_arc_segment_joint0</joint>
+                        <pitch_diameter>${pitch_diameter}</pitch_diameter>
+                    </segment>
+                    <segment>
                         <joint>${name}_straight_segment_joint1</joint>
                     </segment>
                     <segment>
                         <joint>${name}_arc_segment_joint1</joint>
-                        <pitch_diameter>${pitch_diameter}</pitch_diameter>
-                    </segment>
-                    <segment>
-                        <joint>${name}_straight_segment_joint2</joint>
-                    </segment>
-                    <segment>
-                        <joint>${name}_arc_segment_joint2</joint>
                         <pitch_diameter>${pitch_diameter}</pitch_diameter>
                     </segment>
